File: hardware/devboard/cue_devboard.kicad_sch (KiCad schematic)
At the start: 56 parts, among them J1 USB-C (power), J2 BATT, J3 LRA, J4 SWD, J5 EXP, SW1 USER, SW2 SHIP/WAKE, U1 BL54L15, U2 nPM1300, U3 LSM6DSV16BX, U4 T5838, U5 DRV2605L

Commit message: Dev board: Big A's 33 x 21 mm re-layout (v4) plus review fixes
Big A: 35 x 20 mm class layout, J5 replaced by TP11-TP13, BUCK2 removed and
tied off per nPM1300 PS Config 2 (SW2 NC, VSET2 GND, VOUT2 VSYS), fiducials
removed, U3 pin 9 (QVAR2) to GND, USB shield pads on GND.

Review fixes: route U3 pin 9 to a new GND via (it was unconnected on the
board), delete 5 dangling stubs, drop J1's leftover S1 pin (shield is SH).
DRC: 0 unconnected, 0 parity issues; remaining items are courtyard, silk and
thermal-spoke warnings accepted by Big A. fab/bom.csv and cpl.csv are stale.

Co-Authored-By: Claude Opus 5.5 <noreply@anthropic.com>
Parts:
- removed C7: 10uF, Capacitor_SMD:C_0603_1608Metric, symbol Device:C
- removed FID1, FID2, FID3: FID, Fiducial:Fiducial_0.5mm_Mask1mm, symbol Mechanical:Fiducial
- removed J5: EXP, Connector_PinHeader_2.54mm:PinHeader_2x05_P2.54mm_Vertical, symbol Cue:J5
- removed L2: 2.2uH, Inductor_SMD:L_0805_2012Metric, symbol Device:L
- removed R4: 150k, Resistor_SMD:R_0402_1005Metric, symbol Device:R
- removed TP5: TP 3V0, TestPoint:TestPoint_Pad_D1.0mm, symbol Connector:TestPoint
- added TP11, TP12, TP13: TestPoint, TestPoint:TestPoint_Pad_D1.0mm, symbol Connector:TestPoint
Connections:
- net 3V0 is gone; now on net VSYS: U2.32 (VOUT2)
- net EXP_P0_01: now also TP13.1
- net GND: now also J1.SH (SHEILD), U2.16 (VSET2), U3.9 (NC); no longer J1.S1 (GND)
- net PDM_CLK: now also TP11.1
- net PDM_DIN: now also TP12.1
- no-connect marks 31 -> 30
Other:
- moved on the sheet: C1, C10, C11, C12, C16, C17, C18, C19, C2, C20, C21, C22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
